File: MyProjects/MIDI-sync/hardware/MIDI-clock-Eurorack-adapter.kicad_sch (KiCad schematic)
At the start: 24 parts, among them J1 CLOCK, J2 RUN, J3 Conn_02x05_Odd_Even, Q1 2N3904, U1 TL072

Commit message: Update schematic
Parts:
- R7: value 22K -> 10K
Changed lines of the file:
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@@
   (symbol (lib_id "Device:R_US") (at 142.24 162.56 0) (unit 1)
     (in_bom yes) (on_board yes) (dnp no) (fields_autoplaced)
-    (property "Reference" "R7" (at 144.145 161.29 0)
+    (property "Reference" "R7" (at 144.78 161.29 0)
       (effects (font (size 1.27 1.27)) (justify left))
     )
-    (property "Value" "22K" (at 144.145 163.83 0)
+    (property "Value" "10K" (at 144.78 163.83 0)
       (effects (font (size 1.27 1.27)) (justify left))
     )
